File: hw/control_board.brd (EAGLE design)
At the start: 46.7 x 80 mm, 35 parts, among them J1 HD.1-14, Q1 NTD2955G_PCH, Q2 NFET, Q3 NFET_DPAK, Q4 NFET_DPAK, Q5 NFET_DPAK, Q6 NFET_DPAK, U1 BA00BC0WFP-E2_ADJ_LDO, U2 OKI-78SR_3V3_SMPS, U3 AD5290

Commit message: Schematic nearly complete
Parts:
- removed Q2: NFET, pecs:SOT23-3
- added ANT1: PIFA-2.4GHZ, berkeley-epic:PIFA-2.4GHZ
- added C10, C11, C12, C13, C4, C5, C6, C7, C8: 100nF, pecs:0805
- added C9: 10uF, pecs:0805
- added D1, D2, D3, D4, D5: (no value), berkeley-epic:LED-0603
- added IC1: FT232RL, ftdichip:SSOP28
- added J10: ICSP_HDR, pecs:H.1-6
- added J11: HD.1-14, pecs:HD.1-16
- added J12: JTAG, pecs:JTAG
- added J13: HD.1-12, pecs:HD.1-12
- added J8: EPIC-PROG-PORT, berkeley-epic:HEADER2X3X2MM
- added J9: HD.1-6, pecs:HD.1-6
- added R16, R17, R18, R20, R21, R24: 4k7, pecs:0805
- added R22: 10k, pecs:0805
- added R23: 100k, pecs:0805
- added U$1: USB_B, pecs:USB_MOLEX_7041
- added U4: EPIC-CORE_A, berkeley-epic:EPIC-LCC68
- J1: value HD.1-14 -> HD.1-6; device pecs:HD.1-16 -> pecs:HD.1-6
- J7: value (none) -> JTAG; device pecs:H.1-2 -> pecs:JTAG
- Q1: value NTD2955G_PCH -> NFET_DPAK
- R1: value 3k9 -> 10k
- R2: value 33k -> 2k
- R3: value (none) -> 10k
- R4: value (none) -> 100k
- U1: value BA00BC0WFP-E2_ADJ_LDO -> PIC24FJ32GB004; device pecs:TO252-5 -> pecs:TQFP44
- U3: value AD5290 -> NUMONYX_FLASH; device pecs:MSOP10 -> pecs:NUMONYX_FLASH
- moved J1 271.2 mm to (-61.0, -147.3), turned to 0 degrees
- moved J7 218.5 mm to (-61.0, -119.4), turned to 0 degrees
- moved U3 190.1 mm to (-45.7, -101.3)
- moved R4 155.2 mm to (-19.0, -65.6), turned to 0 degrees
- moved R3 118.2 mm to (-19.0, -61.6), turned to 0 degrees
- moved Q1 115.4 mm to (-16.9, -54.1)
- moved R1 108.3 mm to (-4.25, -26.4), turned to 0 degrees
- moved R2 106.8 mm to (-4.25, -30.4), turned to 0 degrees
- moved BLE1 64.8 mm to (25.4, 7.37)
- moved U1 33.8 mm to (56.1, 34.7), turned to 0 degrees
Connections:
- removed net CLK: J1.P13, U3.P6
- removed net FAN_P: J2.P1, J7.P2, Q1.TAG, R1.2, U1.P4
- removed net MOSI: J1.P12, U3.P7
- removed net N$2: R2.2, U3.P2
- removed net N$5: Q1.P1, Q2.P3, R3.1
- removed net POT_CS: J1.P14, U3.P5
- removed net RBYPASS: J1.P11, Q2.P1, R4.2
- removed net UART_MISO: BLE1.P$1, J1.P3
- removed net UART_MOSI: BLE1.P$2, J1.P5
- new net +5V: R24.2, U$1.1_VBUS
- new net ACTL0: J11.P3, U4.P$21
- new net ACTL1: J11.P4, U4.P$22
- new net ACTL2: J11.P5, U4.P$23
- new net ACTL3: J11.P6, U4.P$24
- new net ACTL4: J11.P7, U4.P$25
- new net ACTL5: J11.P8, U4.P$26
- new net AUX_RX: J1.P6, U1.22
- new net AUX_TX: J1.P4, U1.21
- new net BLEGPIO: BLE1.P$27, U4.P$5
- new net BLE_CTS: BLE1.P$3, U1.32
- new net BLE_RTS: BLE1.P$4, U1.31
- new net BLE_RX: BLE1.P$2, U1.11
- new net BLE_TX: BLE1.P$1, U1.5
- new net BL_CTL: J13.P10, U1.3
- new net CMCLR: C10.2, J10.P1, R23.2, U1.18
- new net C_INT0: U1.43, U4.P$20
- new net DCTL0: J11.P9, U4.P$30
- new net DCTL1: J11.P10, U4.P$31
- new net DCTL2: J11.P11, U4.P$32
- new net DCTL3: J11.P12, U4.P$33
- new net E_U1RX: J8.4, U1.15, U4.P$62
- new net E_U1TX: J8.3, U1.14, U4.P$61
- new net FL_CLK: J12.TCK, U1.36, U3.12/6, U3.16
- new net FL_CS: J12.TMS, U1.30, U3.3/1, U3.7
- new net FL_MISO: J12.TDO, U1.38, U3.4/2, U3.8
- new net FL_MOSI: J12.TDI, U1.37, U3.11/5, U3.15
- new net FT_CTS: IC1.11, U1.13
- new net FT_RX: IC1.5, U1.20
- new net FT_TX: IC1.1, U1.19
- new net LCD_EN: Q1.P1, R3.2, U1.41
- new net LCD_GND: J13.P11, Q1.TAG
- new net LCD_RST: J13.P9, U1.35
- new net L_SPI_CLK: J13.P3, U1.25
- new net L_SPI_LCD_CS: J13.P7, U1.23
- new net L_SPI_MISO: J13.P5, U1.27
- new net L_SPI_MOSI: J13.P4, U1.26
- new net L_SPI_TP_CS: J13.P6, U1.24
- new net N$10: D1.C, R16.2
- new net N$11: D2.C, R17.2
- new net N$12: D3.C, R18.2
- new net N$13: R16.1, U4.P$65
- new net N$14: D5.C, R21.2
- new net N$15: R17.1, U4.P$66
- new net N$16: R18.1, U4.P$67
- new net N$17: IC1.22, R20.1
- new net N$18: IC1.23, R21.1
- new net N$19: IC1.19, R22.2, R24.1
- new net N$23: R1.1, R2.2, U4.P$19
- new net N$9: D4.C, R20.2
- new net PGC: J10.P5, U1.9
- new net PGD: J10.P4, U1.8
- new net RH_CLK: J9.P5, U1.44
- new net RH_DAT: J9.P6, U1.1
- new net RST: C8.2, J8.6, R4.2, U4.P$16
- new net TCK: J7.TCK, J8.5, U4.P$15
- new net TDI: J7.TDI, U4.P$13
- new net TDO: J7.TDO, U4.P$12
- new net TMS: J7.TMS, U4.P$14
- new net TP_IRQ: J13.P8, U1.33, U4.P$38
- new net USBD_N: IC1.16, U$1.2_D-
- new net USBD_P: IC1.15, U$1.3_D+
- net +14V: now also J1.P1, J2.P1, R1.2; no longer J7.P1, Q1.P3, R3.2, U1.P1, U1.P2, U3.P9
- net +3V3: now also C11.2, C12.2, C13.2, C4.2, C5.2, C6.2, C7.2, D1.A, D2.A, D3.A, D4.A, D5.A, IC1.20, IC1.4, J1.P2, J10.P2, J11.P1, J11.P14, J12.VDD, J13.P1, J7.VDD, J8.1, J9.P1, R23.1, R4.1, U1.10, U1.17, U1.28, U1.40, U1.42, U3.1, U3.13/7, U3.14/8, U3.2, U3.5/3, U3.9, U4.P$17, U4.P$34, U4.P$37, U4.P$51, U4.P$68; no longer J1.P1
- net FC_A: now also U4.P$6; no longer J1.P4
- net FC_B: now also U4.P$7; no longer J1.P6
- net FC_C: now also U4.P$8; no longer J1.P8
- net GND: now also ANT1.P$2, ANT1.P$3, C10.1, C11.1, C12.1, C13.1, C4.1, C5.1, C6.1, C7.1, C8.1, C9.1, IC1.18, IC1.21, IC1.25, IC1.26, IC1.7, J1.P5, J10.P3, J11.P13, J11.P2, J12.GND, J13.P12, J13.P2, J7.GND, J8.2, J9.P2, Q1.P3, R22.1, R3.1, U$1.4_GND, U1.16, U1.29, U1.39, U1.6, U3.10, U3.6/4, U4.P$1, U4.P$18, U4.P$35, U4.P$42, U4.P$44, U4.P$52; no longer J1.P2, Q2.P2, R4.1, U1.TAG, U3.P3, U3.P4
- net HC: now also U1.2; no longer J1.P10
- net N$1: now also C9.2, U1.7; no longer R1.1, U3.P1
- net N$3: now also ANT1.P$1, U4.P$43; no longer U1.P5, U3.P10
- net RESETB: now also U1.34; no longer J1.P7
- net SYSKEY: now also U1.12; no longer J1.P9
Routing:
- net +14V: track 109.0 -> 0.00 mm, vias 2 -> 0
- net FC_A: track 100.0 -> 0.00 mm
- net FC_B: track 92.8 -> 0.00 mm, vias 1 -> 0
- net HC: track 90.1 -> 0.00 mm, vias 2 -> 0
- net FC_C: track 76.1 -> 0.00 mm, vias 3 -> 0
- net FAN_NEG: track 67.2 -> 0.00 mm, vias 1 -> 0
- net +3V3: track 58.5 -> 0.00 mm, vias 2 -> 0
- net FAN_P: track 45.4 -> 0.00 mm
- net RBYPASS: track 45.2 -> 0.00 mm, vias 2 -> 0
- net CLK: track 39.8 -> 0.00 mm, vias 1 -> 0
- net POT_CS: track 37.3 -> 0.00 mm, vias 2 -> 0
- net N$5: track 36.2 -> 0.00 mm, vias 2 -> 0
- net MOSI: track 35.9 -> 0.00 mm, vias 1 -> 0
- net SYSKEY: track 29.3 -> 0.00 mm, vias 1 -> 0
- net RESETB: track 26.4 -> 0.00 mm, vias 3 -> 0
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- removed copper zone on layer 1, net GND
- removed copper zone on layer 16, net GND
Other:
- board size 46.7 x 80 mm -> 101.6 x 76.2 mm

Commit message: Version 2.0, gerbers rendered
Parts:
- removed Q6: NFET_DPAK, pecs:DPAK
- added Q2: NFET_DPAK, pecs:DPAK
- D1, D2, D3, D4, D5: device berkeley-epic:LED-0603 -> berkeley-epic:LED-1206
- moved J2 184.2 mm to (-82.7, -2.03), turned to 0 degrees
- moved J3 182.3 mm to (-82.8, 47.1), turned to 270 degrees
- moved J11 177.3 mm to (-29.2, 59.4), turned to 90 degrees
- moved J7 176.5 mm to (-62.0, 57.1), turned to 90 degrees
- moved J1 175.4 mm to (-82.8, 26.7)
- moved J4 173.8 mm to (-74.1, 52.1), turned to 90 degrees
- moved ANT1 171.1 mm to (-68.6, 104.3), turned to 90 degrees
- moved J5 169.6 mm to (-74.2, 57.7), turned to 90 degrees
- moved J13 166.7 mm to (-64.9, 27.9)
- moved U3 156.3 mm to (-67.9, 53.5)
- moved IC1 153.2 mm to (-33.8, 22.6), turned to 180 degrees
- moved C10 150.9 mm to (-65.3, 35.0)
- moved R14 150.7 mm to (-54.9, 20.8), turned to 0 degrees
- moved J6 150.1 mm to (-49.2, -2.03), turned to 0 degrees
- moved R5 148.3 mm to (-74.4, -0.76), turned to 270 degrees
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Connections:
- removed net N$17: IC1.22, R20.1
- removed net N$18: IC1.23, R21.1
- new net CB0: IC1.23, R20.1
- new net CB1: IC1.22, R21.1
- net FAN_NEG: now also Q1.TAG; no longer Q4.TAG
- net FC_A: now also Q1.P1; no longer Q4.P1
- net FC_B: now also Q2.P1; no longer Q3.P1
- net FC_C: now also Q3.P1; no longer Q5.P1
- net GND: now also Q2.P3; no longer Q6.P3
- net HC: now also Q4.P1; no longer Q6.P1
- net HEAT_NEG: now also Q4.TAG; no longer Q6.TAG
- net LCD_EN: now also Q5.P1; no longer Q1.P1
- net LCD_GND: now also Q5.TAG; no longer Q1.TAG
- net N$6: now also Q2.TAG; no longer Q3.TAG
- net N$7: now also Q3.TAG; no longer Q5.TAG
Routing:
- net GND: track 0.00 -> 225.0 mm, vias 0 -> 54
- net BLE_RX: track 0.00 -> 130.4 mm, vias 0 -> 2
- net +3V3: track 0.00 -> 116.6 mm, vias 0 -> 19
- net +14V: track 0.00 -> 111.4 mm
- net TP_IRQ: track 0.00 -> 103.1 mm, vias 0 -> 4
- net E_U1RX: track 0.00 -> 87.9 mm, vias 0 -> 2
- net BLE_TX: track 0.00 -> 78.8 mm, vias 0 -> 4
- net E_U1TX: track 0.00 -> 77.7 mm, vias 0 -> 3
- net BLEGPIO: track 0.00 -> 71.7 mm
- net FL_MOSI: track 0.00 -> 66.7 mm, vias 0 -> 2
- net BLE_CTS: track 0.00 -> 62.0 mm, vias 0 -> 2
- net FL_MISO: track 0.00 -> 61.8 mm, vias 0 -> 3
- net FL_CS: track 0.00 -> 61.4 mm, vias 0 -> 2
- net AUX_TX: track 0.00 -> 60.7 mm, vias 0 -> 1
- net BLE_RTS: track 0.00 -> 60.5 mm, vias 0 -> 2
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- added copper zone on layer 15, net +3V3
- added copper zone on layer 1, net GND
- added copper zone on layer 16, net GND
- added copper zone on layer 2, net GND
Other:
- board size 101.6 x 76.2 mm -> 60 x 114 mm
- board text added: "+"
- board text added: "EPIC"
- board text added: "FAN"
- board text added: "FLASH"
- board text added: "HEAT"
- board text added: "ICSP"
- board text added: "M ANDERSEN (C) 2013"
- board text added: "PECS CTL 2.0"
- board text added: "UC BERKELEY"
- board text removed: "(C) 2013 ANDERSEN, BYNOE"
