File: hw/control_board.brd (EAGLE design)
At the start: 46.7 x 80 mm, 35 parts, among them J1 HD.1-14, Q1 NTD2955G_PCH, Q2 NFET, Q3 NFET_DPAK, Q4 NFET_DPAK, Q5 NFET_DPAK, Q6 NFET_DPAK, U1 BA00BC0WFP-E2_ADJ_LDO, U2 OKI-78SR_3V3_SMPS, U3 AD5290

Commit message: joe's v1
Parts:
- moved J1 7.18 mm to (85.3, 72.6)
- moved J4 7.18 mm to (92.7, 72.6)
- moved J5 7.18 mm to (89.2, 72.6)
- moved R11 6.35 mm to (66.3, 2.79)
- moved C2 5.68 mm to (61.7, 54.1)
- moved C1 5.68 mm to (61.7, 71.4)
- moved U2 5.68 mm to (61.7, 62.7)
- moved Q6 3.81 mm to (90.9, 8.13)
- moved R14 3.81 mm to (90.9, 3.05)
- moved U3 3.14 mm to (76.2, 42.7), turned to 270 degrees
- moved BLE1 2.54 mm to (73.7, 48.0)
- moved Q4 2.54 mm to (62.5, 8.13)
- moved Q5 2.54 mm to (81.3, 8.13)
- moved R12 2.54 mm to (75.2, 2.79)
Routing:
- net FC_A: track 100.0 -> 78.8 mm, vias 0 -> 2
- net +3V3: track 58.5 -> 47.4 mm, vias 2 -> 3
- net GND: track 11.1 -> 5.83 mm, vias 2 -> 1
- net +14V: track 109.0 -> 103.9 mm, vias 2 -> 3
- net N$3: track 14.7 -> 10.9 mm, vias 2 -> 0
- net MOSI: track 35.9 -> 32.4 mm
- net HC: track 90.1 -> 87.2 mm
- net FC_B: track 92.8 -> 90.1 mm
- net N$1: track 7.99 -> 10.2 mm, vias 2 -> 0
- net CLK: track 39.8 -> 37.7 mm
- net POT_CS: track 37.3 -> 35.2 mm, vias 2 -> 0
- net RBYPASS: track 45.2 -> 47.2 mm, vias 2 -> 1
- net UART_MISO: track 16.7 -> 18.6 mm, vias 1 -> 0
- net SYSKEY: track 29.3 -> 27.5 mm, vias 1 -> 0
- net RESETB: track 26.4 -> 27.8 mm, vias 3 -> 1
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Other:
- board size 46.7 x 80 mm -> 46.7 x 74.9 mm
