File: hw/control_board.sch (EAGLE design)
At the start: 34 parts, among them J1 HD.1-14, Q1 NTD2955G_PCH, Q2 NFET, Q3 NFET_DPAK, Q4 NFET_DPAK, Q5 NFET_DPAK, Q6 NFET_DPAK, U1 BA00BC0WFP-E2_ADJ_LDO, U2 OKI-78SR_3V3_SMPS, U3 AD5290

Commit message: 2 am on october 29
Parts:
- added C3: 1uF, pecs:0805_CAPACITOR
Connections:
- net FAN_N renamed FAN_NEG
- net HEAT_N renamed HEAT_NEG
- net +3V3: now also C3.P$2
- net GND: now also C3.P$1
Changed lines of the file:
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@@
 <part name="R15" library="pecs" deviceset="0805_RESISTOR" device="" value="4k7"/>
 <part name="FRAME1" library="frames" deviceset="A4L-LOC" device=""/>
+<part name="C3" library="pecs" deviceset="0805_CAPACITOR" device="" value="1uF"/>
+<part name="GND11" library="supply1" deviceset="GND" device=""/>
 </parts>
 <sheets>
@@
 </instance>
 <instance part="FRAME1" gate="G$1" x="-55.88" y="-104.14"/>
+<instance part="C3" gate="G$1" x="-27.94" y="-30.48" smashed="yes" rot="R90">
+<attribute name="NAME" x="-26.162" y="-30.48" size="1.27" layer="95"/>
+<attribute name="VALUE" x="-26.162" y="-32.258" size="1.27" layer="96"/>
+</instance>
+<instance part="GND11" gate="1" x="-27.94" y="-38.1"/>
 </instances>
 <busses>
@@
 <pinref part="BLE1" gate="G$1" pin="VCC"/>
 <wire x1="-12.7" y1="-27.94" x2="-20.32" y2="-27.94" width="0.1524" layer="91"/>
-<wire x1="-20.32" y1="-27.94" x2="-35.56" y2="-27.94" width="0.1524" layer="91"/>
+<wire x1="-20.32" y1="-27.94" x2="-27.94" y2="-27.94" width="0.1524" layer="91"/>
+<wire x1="-27.94" y1="-27.94" x2="-35.56" y2="-27.94" width="0.1524" layer="91"/>
 <wire x1="-35.56" y1="-27.94" x2="-38.1" y2="-25.4" width="0.1524" layer="91"/>
 <pinref part="+3V2" gate="G$1" pin="+3V3"/>
 <pinref part="R15" gate="G$1" pin="P$1"/>
 <junction x="-20.32" y="-27.94"/>
+<pinref part="C3" gate="G$1" pin="P$2"/>
+<junction x="-27.94" y="-27.94"/>
 </segment>
 <segment>
@@
 <label x="83.82" y="-45.72" size="1.27" layer="95"/>
 </segment>
+<segment>
+<pinref part="C3" gate="G$1" pin="P$1"/>
+<pinref part="GND11" gate="1" pin="GND"/>
+<wire x1="-27.94" y1="-33.02" x2="-27.94" y2="-35.56" width="0.1524" layer="91"/>
+</segment>
 </net>
 <net name="FAN_P" class="0">
@@
 </segment>
 </net>
-<net name="FAN_N" class="0">
+<net name="FAN_NEG" class="0">
 <segment>
 <pinref part="Q4" gate="G$1" pin="D"/>
@@
 </segment>
 </net>
-<net name="HEAT_N" class="0">
+<net name="HEAT_NEG" class="0">
 <segment>
 <pinref part="Q6" gate="G$1" pin="D"/>
@@
 </sheet>
 </sheets>
+<errors>
+</errors>
 </schematic>
 </drawing>

Commit message: Schematic nearly complete
Parts:
- removed Q2: NFET, pecs:NFET
- added ANT1: PIFA-2.4GHZ, berkeley-epic:PIFA-2.4GHZ
- added C10, C11, C12, C13, C4, C5, C6, C7, C8: 100nF, pecs:0805_CAPACITOR
- added C9: 10uF, pecs:0805_CAPACITOR
- added D1, D2, D3, D4, D5: (no value), berkeley-epic:LED0603
- added IC1: FT232RL, ftdichip:FT232RL
- added J10: ICSP_HDR, pecs:ICSP_HDR
- added J11: HD.1-14, pecs:HD.1-14
- added J12: JTAG, pecs:JTAG
- added J13: HD.1-12, pecs:HD.1-12
- added J8: EPIC-PROG-PORT, berkeley-epic:EPIC-PROG-PORT
- added J9: HD.1-6, pecs:HD.1-6
- added R16, R17, R18, R20, R21, R24: 4k7, pecs:0805_RESISTOR
- added R22: 10k, pecs:0805_RESISTOR
- added R23: 100k, pecs:0805_RESISTOR
- added U$1: USB_B, pecs:USB_B
- added U4: EPIC-CORE_A, berkeley-epic:EPIC-CORE_A
- J1: value HD.1-14 -> HD.1-6; device pecs:HD.1-14 -> pecs:HD.1-6
- J7: value (none) -> JTAG; device pecs:H.1-2 -> pecs:JTAG
- Q1: value NTD2955G_PCH -> NFET_DPAK; device pecs:NTD2955G_PCH -> pecs:NFET_DPAK
- R1: value 3k9 -> 10k
- R2: value 33k -> 2k
- R3: value (none) -> 10k
- R4: value (none) -> 100k
- U1: value BA00BC0WFP-E2_ADJ_LDO -> PIC24FJ32GB004; device pecs:BA00BC0WFP-E2_ADJ_LDO -> pecs:PIC24FJ32GB004
- U3: value AD5290 -> NUMONYX_FLASH; device pecs:AD5290 -> pecs:NUMONYX_FLASH
Connections:
- removed net CLK: J1.13, U3.CLK
- removed net FAN_P: J2.1, J7.2, Q1.D, R1.P$2, U1.OUT
- removed net MOSI: J1.12, U3.MOSI
- removed net N$2: R2.P$2, U3.B
- removed net N$5: Q1.G, Q2.D, R3.P$1
- removed net POT_CS: J1.14, U3.!CS!
- removed net RBYPASS: J1.11, Q2.G, R4.P$2
- removed net UART_MISO: BLE1.UART_TX, J1.3
- removed net UART_MOSI: BLE1.UART_RX, J1.5
- new net +5V: R24.P$2, U$1.VBUS
- new net ACTL0: J11.3, U4.ADC2
- new net ACTL1: J11.4, U4.ADC3
- new net ACTL2: J11.5, U4.ADC4
- new net ACTL3: J11.6, U4.ADC5
- new net ACTL4: J11.7, U4.ADC6/DAC0
- new net ACTL5: J11.8, U4.ADC7/DAC1
- new net AUX_RX: J1.6, U1.PGEC1/AN3/C2INA/DMH/RP1/PMD1/CN5/RB1
- new net AUX_TX: J1.4, U1.PGED1/AN2/C2INB/DPH/RP0/PMD0/CN4/RB0
- new net BLEGPIO: BLE1.PIO4, U4.P5.3
- new net BLE_CTS: BLE1.UART_CTS, U1.DO/PMA8/RA8
- new net BLE_RTS: BLE1.UART_RTS, U1.OSCO/CLKO/CN29/RA3
- new net BLE_RX: BLE1.UART_RX, U1.AN11/C1INC/RP13/REFO/PMRD/SESSEND/CN13/RB13
- new net BLE_TX: BLE1.UART_TX, U1.RP25/PMA6/CN19/RC9
- new net BL_CTL: J13.10, U1.RP23/PMA0/CN17/RC7
- new net CMCLR: C10.P$2, J10.!RESET!, R23.P$2, U1.!MCLR!
- new net C_INT0: U1.RP7/OMD5/INT0/CN23/RB7, U4.ADC1
- new net DCTL0: J11.9, U4.P1.2
- new net DCTL1: J11.10, U4.P1.5
- new net DCTL2: J11.11, U4.P1.6
- new net DCTL3: J11.12, U4.P1.7
- new net E_U1RX: J8.RX1, U1.AN9/C3INA/VBUSCHG/RP15/VBUSST/CN11/RB15, U4.UART1RX
- new net E_U1TX: J8.TX1, U1.AN10/C3INB/CVREF/VCPCON/VBUSON/RP14/CN12/RB14, U4.UART1TX
- new net FL_CLK: J12.TCK, U1.AN12/RP19/PMBE/CN28/RC3, U3.P_C, U3.S_C
- new net FL_CS: J12.TMS, U1.OSCI/CLKI/C1IND/PMCS1/CN30/RA2, U3.P_!S!, U3.S_!S!
- new net FL_MISO: J12.TDO, U1.RP21/PMA3/CN26/RC5, U3.P_Q, U3.S_Q
- new net FL_MOSI: J12.TDI, U1.RP20/PMA4/CN25/RC4, U3.P_D, U3.S_D
- new net FT_CTS: IC1.!CTS, U1.TCK/PMA7/RA7
- new net FT_RX: IC1.RXD, U1.PGEC3/AN1/C3IND/VREF-/ASCL1/RP6/PMD6/CTED2/SESSVLD/VCMPST2/CN3/RA1
- new net FT_TX: IC1.TXD, U1.PGED3/AN0/C3INC/VREF+/ASDA1/RP5/PMD7/CTED1/VBUSVLD/VCMPST1/CN2/RA0
- new net LCD_EN: Q1.G, R3.P$2, U1.CN27/USBID/RB5
- new net LCD_GND: J13.11, Q1.D
- new net LCD_RST: J13.9, U1.TDI/PMA9/RA9
- new net L_SPI_CLK: J13.3, U1.AN6/RP16/CN8/RC0
- new net L_SPI_LCD_CS: J13.7, U1.AN4/C1INB/DPLN/SDA2/RP2/PMD2/CN6/RB2
- new net L_SPI_MISO: J13.5, U1.AN8/RP18/PMA2/CN10/RC2
- new net L_SPI_MOSI: J13.4, U1.AN7/RP17/CN9/RC1
- new net L_SPI_TP_CS: J13.6, U1.AN5/C1INA/DMLN/RTCC/SCL2/RP3/PMWR/CN7/RB3
- new net N$10: D1.C, R16.P$2
- new net N$11: D2.C, R17.P$2
- new net N$12: D3.C, R18.P$2
- new net N$13: R16.P$1, U4.LED1
- new net N$14: D5.C, R21.P$2
- new net N$15: R17.P$1, U4.LED2
- new net N$16: R18.P$1, U4.LED3
- new net N$17: IC1.CBUS1, R20.P$1
- new net N$18: IC1.CBUS0, R21.P$1
- new net N$19: IC1.!RESET, R22.P$2, R24.P$1
- new net N$23: R1.P$1, R2.P$2, U4.ADC0
- new net N$9: D4.C, R20.P$2
- new net PGC: J10.PGC, U1.PGEC2/D-/VMIO/RP11/CN15/RB11
- new net PGD: J10.PGD, U1.PGED2/D+/VPIO/RP10/CN16/RB10
- new net RH_CLK: J9.5, U1.USBOEN/SCL1/RP8/PMD4/CN22/RB8
- new net RH_DAT: J9.6, U1.SDA1/RP9/PMD3/RCV/CN21/RB9
- new net RST: C8.P$2, J8.RST#, R4.P$2, U4.RST/NMI
- new net TCK: J7.TCK, J8.TCK, U4.TCK
- new net TDI: J7.TDI, U4.TDI/TCLK
- new net TDO: J7.TDO, U4.TDO/TDI
- new net TMS: J7.TMS, U4.TMS
- new net TP_IRQ: J13.8, U1.SOSCI/C2IND/RP4/CN1/RB4, U4.P2.0
- new net USBD_N: IC1.USBDM, U$1.D-
- new net USBD_P: IC1.USBDP, U$1.D+
- net +14V: now also J1.1, J2.1, R1.P$2; no longer J7.1, Q1.S, R3.P$2, U1.CTL, U1.VIN, U3.VDD
- net +3V3: now also C11.P$2, C12.P$2, C13.P$2, C4.P$2, C5.P$2, C6.P$2, C7.P$2, D1.A, D2.A, D3.A, D4.A, D5.A, IC1.VCC, IC1.VCCIO, J1.2, J10.VDD, J11.1, J11.14, J12.VDD, J13.1, J7.VDD, J8.VDD, J9.1, R23.P$1, R4.P$1, U1.AVDD, U1.VBUS, U1.VDD@1, U1.VDD@2, U1.VUSB, U3.P_!HOLD!, U3.P_!W!, U3.P_VCC, U3.S_!HOLD!, U3.S_!W!, U3.S_VCC, U4.AVDD, U4.DVDD, U4.FLASH_WP, U4.FVDD, U4.RVDD; no longer J1.1
- net FC_A: now also U4.P5.4; no longer J1.4
- net FC_B: now also U4.P5.5; no longer J1.6
- net FC_C: now also U4.P5.6; no longer J1.8
- net GND: now also ANT1.RFGND@2, ANT1.RFGND@3, C10.P$1, C11.P$1, C12.P$1, C13.P$1, C4.P$1, C5.P$1, C6.P$1, C7.P$1, C8.P$1, C9.P$1, IC1.GND, IC1.GND@1, IC1.GND@2, IC1.GND@A, IC1.TEST, J1.5, J10.GND, J11.13, J11.2, J12.GND, J13.12, J13.2, J7.GND, J8.GND, J9.2, Q1.S, R22.P$1, R3.P$1, U$1.GND, U1.AVSS, U1.DISVREG, U1.VSS@1, U1.VSS@2, U3.P_VSS, U3.S_VSS, U4.AGND, U4.GND1, U4.GND2, U4.GND3, U4.RFGND1, U4.RFGND2; no longer J1.2, Q2.S, R4.P$1, U1.GND, U3.GND, U3.VSS
- net HC: now also U1.RP22/PMA1/CN18/RC6; no longer J1.10
- net N$1: now also C9.P$2, U1.VCAP/VDDCORE; no longer R1.P$1, U3.A
- net N$3: now also ANT1.RFOUT, U4.RFOUT; no longer U1.ADJ, U3.W
- net RESETB: now also U1.SOSCO/SCLKI/T1CK/C2INC/CN0/RA4; no longer J1.7
- net SYSKEY: now also U1.TMS/PMA10/RA10; no longer J1.9
Other:
- note added: "Bluetooth Low Energy (BLE) Transceiver"
- note added: "Display flash"
- note added: "EPIC core"
- note added: "FLASH SPI"
- note added: "GPIO and display coprocessor"
- note added: "Lowside switching"
- note added: "MODBUS header"
- note added: "MSP430 JTAG"
- note added: "PIC ICSP"
- note added: "PIC24FJ64GB004"
- note added: "Power regulation and decoupling"
- note added: "Programming ports"
- note added: "RH/Temp header"
- note added: "Screen, sensing and actuation headers"
- note added: "UI elements header"
- note added: "USB interface"
- note removed: "Bypass J"
- moved on the sheet: C1, C2, C3, J2, J3, J4, J5, J6, Q1, Q3, Q4, Q5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

Commit message: Version 2.0, gerbers rendered
Parts:
- removed Q6: NFET_DPAK, pecs:NFET_DPAK
- added Q2: NFET_DPAK, pecs:NFET_DPAK
- D1, D2, D3, D4, D5: device berkeley-epic:LED0603 -> berkeley-epic:LED1206
Connections:
- removed net N$17: IC1.CBUS1, R20.P$1
- removed net N$18: IC1.CBUS0, R21.P$1
- new net CB0: IC1.CBUS0, R20.P$1
- new net CB1: IC1.CBUS1, R21.P$1
- net FAN_NEG: now also Q1.D; no longer Q4.D
- net FC_A: now also Q1.G; no longer Q4.G
- net FC_B: now also Q2.G; no longer Q3.G
- net FC_C: now also Q3.G; no longer Q5.G
- net GND: now also Q2.S; no longer Q6.S
- net HC: now also Q4.G; no longer Q6.G
- net HEAT_NEG: now also Q4.D; no longer Q6.D
- net LCD_EN: now also Q5.G; no longer Q1.G
- net LCD_GND: now also Q5.D; no longer Q1.D
- net N$6: now also Q2.D; no longer Q3.D
- net N$7: now also Q3.D; no longer Q5.D
Other:
- note added: "GIT:"
- note added: "Michael Andersen, Joseph Bynoe"
- note added: "PECS CONTROL BOARD"
- note added: "REVISION 1.0 - 12 November 2013"
- moved on the sheet: C1, C10, C11, C12, C13, C2, C4, C5, C6, C7, C9, D4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
